Commit message: working till navigation

File: questbot_description/urdf/2w_diffdrive/body.urdf.xacro (robot description, xacro)
@@ -6,5 +6,5 @@
     <!-- Wheel -->
     <xacro:include filename="macro/wheel.xacro" />
-    <!-- Define robot constants -->
+    <!-- Define robot properties -->
     <!-- Robot base constants -->
     <xacro:property name="base_width" value="0.31" />

File: questbot_description/urdf/2w_diffdrive/control/gazebo_control.xacro (robot description, xacro)
@@ -3,7 +3,4 @@
     <gazebo>
         <plugin name='diff_drive' filename='libgazebo_ros_diff_drive.so'>
-            <ros>
-                <namespace>/demo</namespace>
-            </ros>
             <!-- wheels -->
             <left_joint>left_wheel_joint</left_joint>

File: questbot_description/urdf/2w_diffdrive/gazebo.urdf.xacro (robot description, xacro)
@@ -2,9 +2,9 @@
 <robot xmlns:xacro="http://www.ros.org/wiki/xacro">
     <!-- Properties -->
-    <!-- Choose Gazebo version -->
+    <!-- Gazebo version -->
     <xacro:property name="use_gazebo" value="1" />
     <xacro:property name="use_gzsim" value="0" />
-    <!-- Choose whether to publish odom from controller -->
-    <xacro:property name="publish_odom_tf" value="false"/>
+    <!-- Gazebo properties  -->
+    <xacro:property name="publish_odom_tf" value="true"/>
     <!-- Classic Gazebo -->
     <xacro:if value="$(arg use_gazebo)">

File: questbot_description/urdf/6w_diffdrive/control/gazebo_control.xacro (robot description, xacro)
@@ -1,9 +1,5 @@
-<?xml version="1.0"?>
-<robot xmlns:xacro="http://www.ros.org/wiki/xacro">
+<robot>
     <gazebo>
-        <plugin name='diff_drive' filename='libgazebo_ros_diff_drive.so'>
-            <ros>
-                <namespace>/demo</namespace>
-            </ros>
+        <plugin name="diff_drive" filename="libgazebo_ros_diff_drive.so">
             <!-- wheels -->
             <num_wheel_pairs>3</num_wheel_pairs>
@@ -23,5 +19,5 @@
             <updateRate>100</updateRate>
             <publish_odom>true</publish_odom>
-            <publish_odom_tf>${publish_odom_tf}</publish_odom_tf>
+            <publish_odom_tf>true</publish_odom_tf>
             <publish_wheel_tf>true</publish_wheel_tf>
             <odometry_frame>odom</odometry_frame>
